File: kicad/clocks.kicad_sch (KiCad schematic)
At the start: 39 parts, among them U1 SIT5156A, U2 ICE40LP384-SG32, U3 LMK1C1104, U4 LEA-M8T, U5 TDC7200, U6 LMK1C1104

Commit message: gps bias cap
Parts:
- added C38: 10n, symbol Device:C
Connections:
- net GND: now also C38.2
- net VCC_RF: now also C38.1
Changed lines of the file:
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@@
   (junction (at 69.85 33.02) (diameter 0) (color 0 0 0 0)
+  )
+  (junction (at 299.72 62.23) (diameter 0) (color 0 0 0 0)
   )
   (junction (at 36.83 245.11) (diameter 0) (color 0 0 0 0)
@@
     (stroke (width 0) (type default))
   )
+  (wire (pts (xy 308.61 64.77) (xy 308.61 62.23))
+    (stroke (width 0) (type default))
+  )
   (wire (pts (xy 60.96 33.02) (xy 69.85 33.02))
     (stroke (width 0) (type default))
@@
     (stroke (width 0) (type default))
   )
+  (wire (pts (xy 299.72 62.23) (xy 299.72 67.31))
+    (stroke (width 0) (type default))
+  )
   (wire (pts (xy 347.98 76.2) (xy 347.98 78.74))
     (stroke (width 0) (type default))
@@
     (stroke (width 0) (type default))
   )
+  (wire (pts (xy 308.61 62.23) (xy 299.72 62.23))
+    (stroke (width 0) (type default))
+  )
   (wire (pts (xy 149.86 66.04) (xy 149.86 62.23))
     (stroke (width 0) (type default))
@@
     (stroke (width 0) (type default))
   )
-  (wire (pts (xy 299.72 58.42) (xy 299.72 67.31))
+  (wire (pts (xy 299.72 58.42) (xy 299.72 62.23))
     (stroke (width 0) (type default))
   )
@@
     )
   )
+  (symbol (lib_id "power:GND") (at 308.61 72.39 0) (unit 1)
+    (in_bom yes) (on_board yes) (dnp no) (fields_autoplaced)
+    (property "Reference" "#PWR094" (at 308.61 78.74 0)
+      (effects (font (size 1.27 1.27)) hide)
+    )
+    (property "Value" "GND" (at 308.61 77.47 0)
+      (effects (font (size 1.27 1.27)))
+    )
+    (property "Footprint" "" (at 308.61 72.39 0)
+      (effects (font (size 1.27 1.27)) hide)
+    )
+    (property "Datasheet" "" (at 308.61 72.39 0)
+      (effects (font (size 1.27 1.27)) hide)
+    )
+    (pin "1")
+    (instances
+      (project "gpsrx"
+        (path "/c3c549bc-9d82-4b6a-bdb9-a3870905229d/70e7e3a4-572d-4c59-9c26-94e3cd20e23c"
+          (reference "#PWR094") (unit 1)
+        )
+      )
+    )
+  )
   (symbol (lib_id "bgelb_lib:TDC7200") (at 293.37 204.47 0) (unit 1)
     (in_bom yes) (on_board yes) (dnp no) (fields_autoplaced)
@@
         )
       )
+    )
+  )
+  (symbol (lib_id "Device:C") (at 308.61 68.58 0) (unit 1)
+    (in_bom yes) (on_board yes) (dnp no) (fields_autoplaced)
+    (property "Reference" "C38" (at 312.42 67.31 0)
+      (effects (font (size 1.27 1.27)) (justify left))
+    )
+    (property "Value" "10n" (at 312.42 69.85 0)
+      (effects (font (size 1.27 1.27)) (justify left))
+    )
+    (property "Footprint" "" (at 309.5752 72.39 0)
+      (effects (font (size 1.27 1.27)) hide)
+    )
+    (property "Datasheet" "~" (at 308.61 68.58 0)
+      (effects (font (size 1.27 1.27)) hide)
+    )
+    (pin "1")
+    (pin "2")
+    (instances
+      (project "gpsrx"
+        (path "/c3c549bc-9d82-4b6a-bdb9-a3870905229d/70e7e3a4-572d-4c59-9c26-94e3cd20e23c"
+          (reference "C38") (unit 1)
+        )
+      )

Commit message: bos/tos tweaks
Parts:
- removed R49: 1K, symbol Device:R_US
- added C39: 1u, symbol Device:C
- added U14: TMP117xxDRV, Package_SON:WSON-6-1EP_2x2mm_P0.65mm_EP1x1.6mm, symbol Sensor_Temperature:TMP117xxDRV
Connections:
- net +3.3V: now also C39.1, U14.5 (V+)
- net GND: now also C39.2, U14.2 (GND), U14.4 (ADD0)
- net STOP_BOS_COUNT renamed STOP_TOS_COUNT
- new net SCL_TEMP: U14.1 (SCL)
- new net SDA_TEMP: U14.6 (SDA)
- no-connect marks 16 -> 17
Other:
- note removed: "ADD VCTCXO OPTION HERE"

Commit message: add tcxo
Parts:
- added C40, C42, C45, C46: 1u, symbol Device:C
- added C41: 4.7u, symbol Device:C
- added C43, C44: 2.2u, symbol Device:C
- added R51, R52: 10K, symbol Device:R_US
- added R53, R54: 100K, symbol Device:R_US
- added R55: 0, symbol Device:R_US
- added R56: 1K, symbol Device:R_US
- added U15: OPA376xxDBV, Package_TO_SOT_SMD:SOT-23-5, symbol Amplifier_Operational:OPA376xxDBV
- added U16: AD5689RxRUZ, Package_SO:TSSOP-16_4.4x5mm_P0.65mm, symbol Analog_DAC:AD5689RxRUZ
- added U17: JTP32CSV, symbol bgelb_lib:JTP32CSV
- C1, U1: now not fitted
Connections:
- net +3.3V: now also C40.1, C41.1, C42.1, C45.1, R56.2, U15.5 (V+), U16.11 (VLOGIC), U16.16 (RSTSEL), U16.5 (VDD), U17.4 (Vcc)
- net GND: now also C40.2, C41.2, C42.2, C44.2, C45.2, C46.2, R54.1, U15.2 (V-), U16.10 (GAIN), U16.4 (GND), U16.9 (~{LDAC}), U17.2 (GND)
- net at U1.6 (CLK), U3.1 (CLKIN): now also U17.3 (CLK)
- new net: R51.1, U16.3 (VOUTA)
- new net: R51.2, R54.2, U15.3 (+)
- new net: C46.1, R56.1, U16.15 (~{RESET})
- new net: C43.2, R52.2, R55.1, U15.1
- new net: C43.1, R52.1, R53.2, U15.4 (-)
- new net: R53.1, U16.7 (VOUTB)
- new net: C44.1, R55.2, U17.1 (EFC)
- new net DAC_MISO: U16.8 (SDO)
- new net DAC_MOSI: U16.14 (SDIN)
- new net DAC_SCK: U16.12 (SCLK)
- new net DAC_SS: U16.13 (~{SYNC})
- no-connect marks 17 -> 18
Other:
- note added: "~4.5Hz CUTOFF"
- moved on the sheet: C39, U14

Commit message: add flipflop to stop path
Parts:
- added C47: 1u, symbol Device:C
- added U18: 74AUC1G79, symbol 74xGxx:74AUC1G79
- R51, R52: value 10K -> 2K
Connections:
- net +3.3V: now also C47.1, U18.5 (VCC)
- net CLK_TDC: now also U18.2 (C)
- net GND: now also C47.2, U18.3 (GND)
- net TDC_STOP: now also U18.4 (Q); no longer U2.23 (IOR_39)
- net DAC_COARSE: now reaches R51.1, U16.3 (VOUTA)
- net OPA_FF: now reaches R51.2, R54.2, U15.3 (+)
- net DAC_RESET: now reaches C46.1, R56.1, U16.15 (~{RESET})
- net EFC: now reaches C43.2, R52.2, R55.1, U15.1
- net OPA_FB: now reaches C43.1, R52.1, R53.2, U15.4 (-)
- net DAC_FINE: now reaches R53.1, U16.7 (VOUTB)
- net EFC_FILT: now reaches C44.1, R55.2, U17.1 (EFC)
- net GPS_MISO_R: now reaches R6.2, U4.3 (TXD/SPI_MISO)
- new net TDC_STOP_NEXT: U18.1 (D), U2.23 (IOR_39)
Other:
- note added: "EFC CENTER VOLTAGE = 1.5V TUNING RANGE +/- 1V =~ +/- 10PPM OSC SPEC 280PPB OVER -40C to +85C V_EFC = (-0.02)V_DAC_FINE + V_DAC_COARSE GIVES +/- 0.02V => +/- 200PPB FINE TUNING RANGE"
- note added: "PLACE NEAR OSCILLATORS"

Commit message: add flop to pps out
Parts:
- added C48: 1u, symbol Device:C
- added R61: 22, symbol Device:R_US
- added U19: 74AUC1G79, symbol 74xGxx:74AUC1G79
- C44: value 2.2u -> 100u; now fitted
- R13, R16, R2, R4, R5: value 22 -> 0
- R55: value 0 -> 1K
Connections:
- net +3.3V: now also C48.1, U19.5 (VCC)
- net GND: now also C48.2, U19.3 (GND)
- net PPS_CLEAN_OUT: now also R61.2; no longer U2.1 (IOL_2B)
- net at R3.1, U3.7 (Y3): now also U19.2 (C)
- new net: R61.1, U19.4 (Q)
- new net PPS_CLEAN_NEXT: U19.1 (D), U2.1 (IOL_2B)
Other:
- moved on the sheet: C1, C2, C39, C47, C5, C6, R1, R12, R15, R2, R3, R4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

Commit message: power and frontend updates
Connections:
- net +3.3V: no longer C1.1, C10.1, C11.1, C12.1, C13.1, C2.1, C41.1, C42.1, C45.1, C48.1, C9.1, R1.1, R56.2, U1.9 (VDD), U15.5 (V+), U16.5 (VDD), U17.4 (Vcc), U19.5 (VCC), U2.16 (VCC_SPI), U2.17 (VCCIO_1), U2.28 (VCCIO_0), U2.4 (VCCIO_3), U2.9 (VCCIO_2), U3.6 (VDD)
- new net +3.3VA: C1.1, C2.1, C41.1, C42.1, C45.1, C48.1, R1.1, R56.2, U1.9 (VDD), U15.5 (V+), U16.5 (VDD), U17.4 (Vcc), U19.5 (VCC), U3.6 (VDD)
- new net +3.3VP: C10.1, C11.1, C12.1, C13.1, C9.1, U2.16 (VCC_SPI), U2.17 (VCCIO_1), U2.28 (VCCIO_0), U2.4 (VCCIO_3), U2.9 (VCCIO_2)

Commit message: swap ice40 for max v, add 1.2v switcher
Parts:
- removed C15: 4.7u, symbol Device:C
- removed R12: 22, symbol Device:R_US
- removed U2: ICE40LP384-SG32, QFNS32_LAT, symbol bgelb_lib:ICE40LP384-SG32
- added R88, R89: 10K, symbol Device:R_US
- added R90: 1K, symbol Device:R_US
- added U2: 5M160ZE64, bgelb_footprint:EQFP64_A-1P20_D2-4P5_INT, symbol bgelb_lib:5M160ZE64
- R18: now not fitted
Connections:
- net +3.3V: now also C10.1, C11.1, C12.1, C9.1, R88.1, R89.1, U2.23 (VCCIO1), U2.39 (VCCIO2), U2.57 (VCCIO2), U2.6 (VCCIO1)
- net CLK_TF: now also U2.7 (IO_CLK0)
- net CLK_UC: now also U2.38 (IO)
- net GND: now also R90.2, U2.28 (IO_DEV_OE_B5_P), U2.29 (IO_DEV_CLRN_B5_N), U2.65 (GND)
- net PPS_CLEAN_NEXT: now also U2.36 (IO_R3_N)
- net PPS_CLEAN_UC: now also U2.37 (IO_R3_P)
- net PPS_RAW_LOGIC: now also U2.5 (IO)
- net STOP_TOS_COUNT: now also U2.43 (IO_R2_N)
- net TDC_STOP_NEXT: now also U2.44 (IO_R2_P)
- net TF_MISO_OUT: now also U2.10 (IO)
- net TF_MOSI: now also U2.11 (IO_L3_P)
- net TF_RESET_L: now also U2.1 (IO_L1_N)
- net TF_SCK: now also U2.13 (IO)
- net TF_SS: now also U2.12 (IO_L3_N)
- net TOS_MARK_DDC: now also U2.48 (IO)
- net +2V5 renamed +1V8
- net +1V8: now also C13.1, U2.41 (VCCINT), U2.8 (VCCINT)
- removed net +3.3VP: C10.1, C11.1, C12.1, C13.1, C9.1
- net TDC_INTB_OUT: no longer names the net of U5.8 (INTB)
- new net STOP_DONE: U2.42 (IO_CLK3)
- new net TF_TCK: R90.1, U2.16 (TCK)
- new net TF_TDI: R89.2, U2.15 (TDI)
- new net TF_TDO: U2.17 (TDO)
- new net TF_TMS: R88.2, U2.14 (TMS)
- no-connect marks 18 -> 9
Other:
- note removed: "UC CONFIGURES FPGA VIA SPI SLAVE MODE"
- moved on the sheet: C10, C11, C12, C9

Commit message: add lte radio and various fixes
Parts:
- R13, R4: value 0 -> 22
Connections:
- net UC_CLK: now reaches U2.40 (IO_CLK2)
- net CLK_UC renamed UC_SLOW_CLOCK
- net PPS_CLEAN_UC renamed UC_PPS_NEXT
- net PPS_RAW_LOGIC renamed PPS_RAW_TF
- net STOP_DONE renamed UC_STOP_DONE
- net STOP_TOS_COUNT renamed UC_STOP_NEXT
Changed lines of the file:
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@@
+    (stroke (width 0) (type default))
+  )
+  (wire (pts (xy 170.18 212.09) (xy 185.42 212.09))
     (stroke (width 0) (type default))
   )
@@
     )
   )
-  (global_label "PPS_RAW_LOGIC" (shape output) (at 388.62 59.69 0) (fields_autoplaced)
+  (global_label "PPS_RAW_TF" (shape output) (at 388.62 59.69 0) (fields_autoplaced)
     (effects (font (size 1.27 1.27)) (justify left))
-    (property "Intersheetrefs" "${INTERSHEET_REFS}" (at 406.6033 59.69 0)
+    (property "Intersheetrefs" "${INTERSHEET_REFS}" (at 403.1561 59.69 0)
       (effects (font (size 1.27 1.27)) (justify left) hide)
     )
@@
     )
   )
-  (global_label "STOP_DONE" (shape output) (at 181.61 209.55 0) (fields_autoplaced)
+  (global_label "UC_STOP_DONE" (shape output) (at 181.61 209.55 0) (fields_autoplaced)
     (effects (font (size 1.27 1.27)) (justify left))
-    (property "Intersheetrefs" "${INTERSHEET_REFS}" (at 195.4204 209.55 0)
-      (effects (font (size 1.27 1.27)) (justify left) hide)
-    )
-  )
-  (global_label "PPS_RAW_LOGIC" (shape input) (at 88.9 207.01 180) (fields_autoplaced)
-    (effects (font (size 1.27 1.27)) (justify right))
-    (property "Intersheetrefs" "${INTERSHEET_REFS}" (at 70.9167 207.01 0)
+    (property "Intersheetrefs" "${INTERSHEET_REFS}" (at 198.9885 209.55 0)
+      (effects (font (size 1.27 1.27)) (justify left) hide)
+    )
+  )
+  (global_label "PPS_RAW_TF" (shape input) (at 88.9 207.01 180) (fields_autoplaced)
+    (effects (font (size 1.27 1.27)) (justify right))
+    (property "Intersheetrefs" "${INTERSHEET_REFS}" (at 74.3639 207.01 0)
       (effects (font (size 1.27 1.27)) (justify right) hide)
     )
@@
     )
   )
-  (global_label "STOP_TOS_COUNT" (shape output) (at 181.61 207.01 0) (fields_autoplaced)
+  (global_label "UC_STOP_NEXT" (shape output) (at 181.61 207.01 0) (fields_autoplaced)
     (effects (font (size 1.27 1.27)) (justify left))
-    (property "Intersheetrefs" "${INTERSHEET_REFS}" (at 201.0447 207.01 0)
+    (property "Intersheetrefs" "${INTERSHEET_REFS}" (at 198.5651 207.01 0)
       (effects (font (size 1.27 1.27)) (justify left) hide)
     )
@@
     )
   )
-  (global_label "CLK_UC" (shape output) (at 185.42 214.63 0) (fields_autoplaced)
+  (global_label "UC_SLOW_CLOCK" (shape output) (at 185.42 214.63 0) (fields_autoplaced)
     (effects (font (size 1.27 1.27)) (justify left))
-    (property "Intersheetrefs" "${INTERSHEET_REFS}" (at 195.5414 214.63 0)
+    (property "Intersheetrefs" "${INTERSHEET_REFS}" (at 204.129 214.63 0)
       (effects (font (size 1.27 1.27)) (justify left) hide)
     )
@@
     (property "Intersheetrefs" "${INTERSHEET_REFS}" (at 60.152 219.71 0)
       (effects (font (size 1.27 1.27)) (justify right) hide)
+    )
+  )
+  (global_label "UC_CLK" (shape output) (at 185.42 212.09 0) (fields_autoplaced)
+    (effects (font (size 1.27 1.27)) (justify left))
+    (property "Intersheetrefs" "${INTERSHEET_REFS}" (at 195.5414 212.09 0)
+      (effects (font (size 1.27 1.27)) (justify left) hide)
     )
   )
@@
     )
   )
-  (global_label "PPS_CLEAN_UC" (shape output) (at 185.42 217.17 0) (fields_autoplaced)
+  (global_label "UC_PPS_NEXT" (shape output) (at 185.42 217.17 0) (fields_autoplaced)
     (effects (font (size 1.27 1.27)) (justify left))
-    (property "Intersheetrefs" "${INTERSHEET_REFS}" (at 202.5566 217.17 0)
+    (property "Intersheetrefs" "${INTERSHEET_REFS}" (at 201.347 217.17 0)
       (effects (font (size 1.27 1.27)) (justify left) hide)
     )
@@
       (effects (font (size 1.27 1.27)))
     )
-    (property "Value" "0" (at 135.89 54.61 90)
+    (property "Value" "22" (at 135.89 54.61 90)
       (effects (font (size 1.27 1.27)))
     )
@@
       (effects (font (size 1.27 1.27)))
     )
-    (property "Value" "0" (at 375.92 67.31 90)
-      (effects (font (size 1.27 1.27)))
-    )
+    (property "Value" "22" (at 375.92 67.31 90)
+      (effects (font (size 1.27 1.27)))
+    )
