File: kicad/clocks.kicad_sch (KiCad schematic)
At the start: 63 parts, among them U1 SIT5156A, U14 TMP117xxDRV, U15 OPA376xxDBV, U16 AD5689RxRUZ, U17 JTP32CSV, U18 74AUC1G79, U19 74AUC1G79, U2 5M160ZE64, U3 LMK1C1104, U4 LEA-M8T, U5 TDC7200, U6 LMK1C1104

Commit message: assign footprints
Parts:
- BT1: footprint (none) -> Battery:Battery_Panasonic_CR1025-VSK_Vertical_CircularHoles
- C1, C10, C11, C12, C13, C14, C2, C3, C38, C39, C4, C40, C41, C42, C43, C45, C46, C47, C48, C5, C6, C9: footprint (none) -> Capacitor_SMD:C_0603_1608Metric_Pad1.08x0.95mm_HandSolder
- C44: footprint (none) -> Capacitor_SMD:C_1206_3216Metric_Pad1.33x1.80mm_HandSolder
- R1, R10, R11, R13, R14, R15, R16, R17, R18, R2, R3, R4, R5, R51, R52, R53, R54, R55, R56, R6, R61, R7, R8, R88, R89, R9, R90: footprint (none) -> Resistor_SMD:R_0603_1608Metric_Pad0.98x0.95mm_HandSolder
- U1: footprint (none) -> bgelb_footprint:CQFN10L_5.000X3.200X0.950_SIT
- U17: footprint (none) -> Oscillator:Oscillator_SMD_Abracon_ASE-4Pin_3.2x2.5mm_HandSoldering
- U18, U19: footprint (none) -> Package_TO_SOT_SMD:SOT-23-5_HandSoldering
- U3, U6: footprint (none) -> Package_SO:TSSOP-8_4.4x3mm_P0.65mm
- U4: footprint RF_GPS:ublox_LEA -> bgelb_footprint:SMT_M8T-0_UBL
- U5: footprint (none) -> Package_SO:TSSOP-14_4.4x5mm_P0.65mm
Connections:
- no-connect marks 9 -> 46

Commit message: fix ercs
Parts:
- added R126, R127: 0, Resistor_SMD:R_0603_1608Metric_Pad0.98x0.95mm_HandSolder, symbol Device:R_US
- added R128, R129: 1K, Resistor_SMD:R_0603_1608Metric_Pad0.98x0.95mm_HandSolder, symbol Device:R_US
Connections:
- net GND: now also R128.2, R129.2; no longer U2.28 (IO_DEV_OE_B5_P), U2.29 (IO_DEV_CLRN_B5_N)
- net PPS_CLEAN_R: now also R61.1, U19.4 (Q)
- new net: R126.2, R127.2, U3.1 (CLKIN)
- new net: R129.1, U2.29 (IO_DEV_CLRN_B5_N)
- new net: R128.1, U2.28 (IO_DEV_OE_B5_P)
- new net: R126.1, U1.6 (CLK)
- new net: R127.1, U17.3 (CLK)
- no-connect marks 46 -> 47

Commit message: add net names
Parts:
- removed R15, R6: 0, Resistor_SMD:R_0603_1608Metric_Pad0.98x0.95mm_HandSolder, symbol Device:R_US
Connections:
- net GPS_MISO_R is gone; now on net GPS_MISO: U4.3 (TXD/SPI_MISO)
- net TDC_MISO_OUT is gone; now on net TDC_MISO: U5.9 (DOUT)
- net LO_CLKEN: now reaches R1.2, U3.2 (1G)
- net LO_CLKOUT: now reaches R126.2, R127.2, U3.1 (CLKIN)
- net CLK_TDC_R: now reaches R4.1, U3.3 (Y0)
- net CLK_DDC_R: now reaches R5.1, U3.5 (Y2)
- net CLK_OUT_R: now reaches R3.1, U19.2 (C), U3.7 (Y3)
- net CLK_TF_R: now reaches R2.1, U3.8 (Y1)
- net SIT_CLKOUT: now reaches R126.1, U1.6 (CLK)
- net PPS_RAW_EN: now reaches R11.2, U6.2 (1G)
- net XO_CLKOUT: now reaches R127.1, U17.3 (CLK)
- net RAW_OUT_R: now reaches R14.1, U6.7 (Y3)
- net RAW_TF_R: now reaches R16.1, U6.3 (Y0)
- net RAW_UC_R: now reaches R17.1, U6.5 (Y2)
- net RAW_TDC_R: now reaches R13.1, U6.8 (Y1)
Other:
- moved on the sheet: R1, R11, R126, R127
