File: kicad/gpsrx.kicad_sch (KiCad schematic)
At the start: 0 parts

Commit message: updates
Other:
- added sheet RF Frontend (rf_frontend.kicad_sch)
Changed lines of the file:
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@@
+    )
+  )
+  (sheet (at 358.14 96.52) (size 31.75 6.35) (fields_autoplaced)
+    (stroke (width 0.1524) (type solid))
+    (fill (color 0 0 0 0.0000))
+    (property "Sheetname" "RF Frontend" (at 358.14 95.8084 0)
+      (effects (font (size 1.27 1.27)) (justify left bottom))
+    )
+    (property "Sheetfile" "rf_frontend.kicad_sch" (at 358.14 103.4546 0)
+      (effects (font (size 1.27 1.27)) (justify left top))
+    )
+    (instances
+      (project "gpsrx"
+        (path "/c3c549bc-9d82-4b6a-bdb9-a3870905229d" (page "5"))
+      )
     )
   )

Commit message: updates
Other:
- added sheet DDC FPGA (ddc_fpga.kicad_sch)
- added sheet MCU (mcu.kicad_sch)
Changed lines of the file:
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@@
+    )
+  )
+  (sheet (at 330.2 185.42) (size 43.18 3.81) (fields_autoplaced)
+    (stroke (width 0.1524) (type solid))
+    (fill (color 0 0 0 0.0000))
+    (property "Sheetname" "DDC FPGA" (at 330.2 184.7084 0)
+      (effects (font (size 1.27 1.27)) (justify left bottom))
+    )
+    (property "Sheetfile" "ddc_fpga.kicad_sch" (at 330.2 189.8146 0)
+      (effects (font (size 1.27 1.27)) (justify left top))
+    )
+    (instances
+      (project "gpsrx"
+        (path "/c3c549bc-9d82-4b6a-bdb9-a3870905229d" (page "7"))
+      )
+    )
+  )
+  (sheet (at 323.85 162.56) (size 39.37 3.81) (fields_autoplaced)
+    (stroke (width 0.1524) (type solid))
+    (fill (color 0 0 0 0.0000))
+    (property "Sheetname" "MCU" (at 323.85 161.8484 0)
+      (effects (font (size 1.27 1.27)) (justify left bottom))
+    )
+    (property "Sheetfile" "mcu.kicad_sch" (at 323.85 166.9546 0)
+      (effects (font (size 1.27 1.27)) (justify left top))
+    )
+    (instances
+      (project "gpsrx"
+        (path "/c3c549bc-9d82-4b6a-bdb9-a3870905229d" (page "6"))
+      )
     )
   )

Commit message: add lte radio and various fixes
Other:
- added sheet LTE Radio (lte_radio.kicad_sch)
Changed lines of the file:
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@@
+    )
+  )
+  (sheet (at 127 142.24) (size 52.07 10.16) (fields_autoplaced)
+    (stroke (width 0.1524) (type solid))
+    (fill (color 0 0 0 0.0000))
+    (property "Sheetname" "LTE Radio" (at 127 141.5284 0)
+      (effects (font (size 1.27 1.27)) (justify left bottom))
+    )
+    (property "Sheetfile" "lte_radio.kicad_sch" (at 127 152.9846 0)
+      (effects (font (size 1.27 1.27)) (justify left top))
+    )
+    (instances
+      (project "gpsrx"
+        (path "/c3c549bc-9d82-4b6a-bdb9-a3870905229d" (page "8"))
+      )
     )
   )
